Commit message: Update xml

File: rmcs_ws/src/rmcs_description/urdf/common.xacro (robot description, xacro)
@@ -6,5 +6,6 @@
       <mass value="${mass}" />
       <xacro:insert_block name="origin" />
-      <inertia ixx="${2.0/5 * mass * radius * radius}" ixy="0.0" ixz="0.0" iyy="${2.0/5 * mass * radius * radius}" iyz="0.0" izz="${2.0/5 * mass * radius * radius}" />
+      <inertia ixx="${2.0/5 * mass * radius * radius}" ixy="0.0" ixz="0.0"
+        iyy="${2.0/5 * mass * radius * radius}" iyz="0.0" izz="${2.0/5 * mass * radius * radius}" />
     </inertial>
   </xacro:macro>
@@ -13,5 +14,7 @@
       <mass value="${mass}" />
       <xacro:insert_block name="origin" />
-      <inertia ixx="${1.0/12 * mass * (3 * radius * radius + length * length)}" ixy="0.0" ixz="0.0" iyy="${1.0/12 * mass * (3 * radius * radius + length * length)}" iyz="0.0" izz="${1.0/2 * mass * radius * radius}" />
+      <inertia ixx="${1.0/12 * mass * (3 * radius * radius + length * length)}" ixy="0.0" ixz="0.0"
+        iyy="${1.0/12 * mass * (3 * radius * radius + length * length)}" iyz="0.0"
+        izz="${1.0/2 * mass * radius * radius}" />
     </inertial>
   </xacro:macro>
@@ -20,5 +23,6 @@
       <mass value="${mass}" />
       <xacro:insert_block name="origin" />
-      <inertia ixx="${1.0/12 * mass * (y*y + z*z)}" ixy="0.0" ixz="0.0" iyy="${1.0/12 * mass * (x*x + z*z)}" iyz="0.0" izz="${1.0/12 * mass * (x*x + y*y)}" />
+      <inertia ixx="${1.0/12 * mass * (y*y + z*z)}" ixy="0.0" ixz="0.0"
+        iyy="${1.0/12 * mass * (x*x + z*z)}" iyz="0.0" izz="${1.0/12 * mass * (x*x + y*y)}" />
     </inertial>
   </xacro:macro>
@@ -27,5 +31,9 @@
       <mass value="${mass}" />
       <xacro:insert_block name="origin" />
-      <inertia ixx="${(-3*h*h*h/20+3*h*h*r/4-4*h*r*r/3+r*r*r)*3*mass/(3*r-h)+(3/4*(h-2*r)*(h-2*r)/(3*r-h))*(3/4*(h-2*r)*(h-2*r)/(3*r-h))}" ixy="0.0" ixz="0.0" iyy="${(-3*h*h*h/20+3*h*h*r/4-4*h*r*r/3+r*r*r)*3*mass/(3*r-h)+(3/4*(h-2*r)*(h-2*r)/(3*r-h))*(3/4*(h-2*r)*(h-2*r)/(3*r-h))}" iyz="0.0" izz="${mass*h/(10*(3*r-h))*(3*h*h-15*h*r+20*r*r)}" />
+      <inertia
+        ixx="${(-3*h*h*h/20+3*h*h*r/4-4*h*r*r/3+r*r*r)*3*mass/(3*r-h)+(3/4*(h-2*r)*(h-2*r)/(3*r-h))*(3/4*(h-2*r)*(h-2*r)/(3*r-h))}"
+        ixy="0.0" ixz="0.0"
+        iyy="${(-3*h*h*h/20+3*h*h*r/4-4*h*r*r/3+r*r*r)*3*mass/(3*r-h)+(3/4*(h-2*r)*(h-2*r)/(3*r-h))*(3/4*(h-2*r)*(h-2*r)/(3*r-h))}"
+        iyz="0.0" izz="${mass*h/(10*(3*r-h))*(3*h*h-15*h*r+20*r*r)}" />
       <origin></origin>
     </inertial>
@@ -35,11 +43,16 @@
       <mass value="${mass}" />
       <xacro:insert_block name="origin" />
-      <inertia ixx="${mass/20*(20*h*h*h*r-10*h*h*h*t-60*h*h*r*r+30*h*h*r*t+120*h*r*r*r-120*h*r*r*t+60*h*r*t*t-15*h*t*t*t-60*r*r*r*t+100*r*r*t*t-65*r*t*t*t+16*t*t*t*t)/(2*t*t*-3*r*t-3*h*t+6*h*r)+(3/4*(t-2*r)*(2*r*r-4*r*r+2*r*t-t*t)/(6*r*r-3*r*t-3*r*t+2*t*t))*(3/4*(t-2*r)*(2*r*r-4*r*r+2*r*t-t*t)/(6*r*r-3*r*t-3*r*t+2*t*t))}" ixy="0.0" ixz="0.0" iyy="${mass/20*(20*h*h*h*r-10*h*h*h*t-60*h*h*r*r+30*h*h*r*t+120*h*r*r*r-120*h*r*r*t+60*h*r*t*t-15*h*t*t*t-60*r*r*r*t+100*r*r*t*t-65*r*t*t*t+16*t*t*t*t)/(2*t*t*-3*r*t-3*h*t+6*h*r)+(3/4*(t-2*r)*(2*r*r-4*r*r+2*r*t-t*t)/(6*r*r-3*r*t-3*r*t+2*t*t))*(3/4*(t-2*r)*(2*r*r-4*r*r+2*r*t-t*t)/(6*r*r-3*r*t-3*r*t+2*t*t))}" iyz="0.0" izz="${mass/(10*(2*t*t-3*r*t-3*h*t+6*h*r))*(-20*h*h*h*r+10*h*h*h*t+60*h*h*r*r-30*h*h*r*t-60*h*r*r*t+60*h*r*t*t-15*h*t*t*t+20*r*r*t*t-25*r*t*t*t+8*t*t*t*t)}" />
+      <inertia
+        ixx="${mass/20*(20*h*h*h*r-10*h*h*h*t-60*h*h*r*r+30*h*h*r*t+120*h*r*r*r-120*h*r*r*t+60*h*r*t*t-15*h*t*t*t-60*r*r*r*t+100*r*r*t*t-65*r*t*t*t+16*t*t*t*t)/(2*t*t*-3*r*t-3*h*t+6*h*r)+(3/4*(t-2*r)*(2*r*r-4*r*r+2*r*t-t*t)/(6*r*r-3*r*t-3*r*t+2*t*t))*(3/4*(t-2*r)*(2*r*r-4*r*r+2*r*t-t*t)/(6*r*r-3*r*t-3*r*t+2*t*t))}"
+        ixy="0.0" ixz="0.0"
+        iyy="${mass/20*(20*h*h*h*r-10*h*h*h*t-60*h*h*r*r+30*h*h*r*t+120*h*r*r*r-120*h*r*r*t+60*h*r*t*t-15*h*t*t*t-60*r*r*r*t+100*r*r*t*t-65*r*t*t*t+16*t*t*t*t)/(2*t*t*-3*r*t-3*h*t+6*h*r)+(3/4*(t-2*r)*(2*r*r-4*r*r+2*r*t-t*t)/(6*r*r-3*r*t-3*r*t+2*t*t))*(3/4*(t-2*r)*(2*r*r-4*r*r+2*r*t-t*t)/(6*r*r-3*r*t-3*r*t+2*t*t))}"
+        iyz="0.0"
+        izz="${mass/(10*(2*t*t-3*r*t-3*h*t+6*h*r))*(-20*h*h*h*r+10*h*h*h*t+60*h*h*r*r-30*h*h*r*t-60*h*r*r*t+60*h*r*t*t-15*h*t*t*t+20*r*r*t*t-25*r*t*t*t+8*t*t*t*t)}" />
     </inertial>
   </xacro:macro>
   <xacro:macro name="default_inertial">
     <inertial>
-      <mass value="0.01"/>
-      <origin xyz="0 0 0"/>
+      <mass value="0.01" />
+      <origin xyz="0 0 0" />
       <inertia ixx="0.001" ixy="0.0" ixz="0.0" iyy="0.001" iyz="0.0" izz="0.001" />
     </inertial>

File: rmcs_ws/src/rmcs_description/urdf/rmcs.urdf.xacro (robot description, xacro)
@@ -8,6 +8,6 @@
   <xacro:arg name="sim_gazebo" default="false" />
   <xacro:arg name="simulation_controllers" default="" />
-  <xacro:include filename="$(find rmcs_description)/urdf/rmcs/rmcs_macro.xacro"/>
-  <xacro:include filename="$(find rmcs_description)/urdf/rmcs/rmcs_macro.ros2_control.xacro"/>
+  <xacro:include filename="$(find rmcs_description)/urdf/rmcs/rmcs_macro.xacro" />
+  <xacro:include filename="$(find rmcs_description)/urdf/rmcs/rmcs_macro.ros2_control.xacro" />
   <!-- create link fixed to the "world" -->
   <link name="world" />
@@ -18,4 +18,11 @@
     <!-- position robot in the world -->
   </xacro:rmcs>
-  <xacro:rmcs_ros2_control name="rmcs" prefix="$(arg prefix)" use_mock_hardware="$(arg use_mock_hardware)" mock_sensor_commands="$(arg mock_sensor_commands)" sim_gazebo_classic="$(arg sim_gazebo_classic)" sim_gazebo="$(arg sim_gazebo)" simulation_controllers="$(arg simulation_controllers)" />
+  <xacro:rmcs_ros2_control
+    name="rmcs"
+    prefix="$(arg prefix)"
+    use_mock_hardware="$(arg use_mock_hardware)"
+    mock_sensor_commands="$(arg mock_sensor_commands)"
+    sim_gazebo_classic="$(arg sim_gazebo_classic)"
+    sim_gazebo="$(arg sim_gazebo)"
+    simulation_controllers="$(arg simulation_controllers)" />
 </robot>

File: rmcs_ws/src/rmcs_description/urdf/rmcs/rmcs_macro.ros2_control.xacro (robot description, xacro)
@@ -1,8 +1,12 @@
 <?xml version="1.0" encoding="UTF-8"?>
 <robot xmlns:xacro="http://wiki.ros.org/xacro">
-  <xacro:macro name="rmcs_ros2_control" params="
-               name
-               prefix use_mock_hardware:=^|false mock_sensor_commands:=^|false sim_gazebo_classic:=^|false sim_gazebo:=^|false
-               simulation_controllers">
+  <xacro:macro name="rmcs_ros2_control"
+    params="name
+            prefix
+            use_mock_hardware:=^|false
+            mock_sensor_commands:=^|false
+            sim_gazebo_classic:=^|false
+            sim_gazebo:=^|false
+            simulation_controllers">
     <ros2_control name="${name}" type="system">
       <hardware>
@@ -31,8 +35,8 @@
         <state_interface name="position">
           <param name="initial_value">0.0</param>
-          <param name="min">0</param>
-          <param name="max">8191</param>
+          <param name="min">0.0</param>
+          <param name="max">8191.0</param>
         </state_interface>
-        <state_interface name="velocity"/>
+        <state_interface name="velocity" />
       </joint>
     </ros2_control>
@@ -52,5 +56,6 @@
       </gazebo>
       <gazebo>
-        <plugin filename="libign_ros2_control-system.so" name="ign_ros2_control::IgnitionROS2ControlPlugin">
+        <plugin filename="libign_ros2_control-system.so"
+          name="ign_ros2_control::IgnitionROS2ControlPlugin">
           <parameters>${simulation_controllers}</parameters>
           <controller_manager_node_name>${prefix}controller_manager</controller_manager_node_name>

File: rmcs_ws/src/rmcs_description/urdf/rmcs/rmcs_macro.xacro (robot description, xacro)
@@ -8,10 +8,10 @@
       <!-- Default inertial for Gazebo/Ingnition - copy and edit block from 'common.xacro'
            to get more realistic behaviour-->
-      <xacro:default_inertial/>
+      <xacro:default_inertial />
       <visual>
         <origin xyz="0 0 0" rpy="0 0 0" />
         <geometry>
           <cylinder length="0.3" radius="0.3" />
-          <!--           <mesh filename="package://rmcs_description/meshes/rmcs/visual/base_link.dae" /> -->
+          <!-- <mesh filename="package://rmcs_description/meshes/rmcs/visual/base_link.dae" /> -->
         </geometry>
       </visual>
@@ -20,9 +20,9 @@
         <geometry>
           <cylinder length="0.3" radius="0.3" />
-          <!--           <mesh filename="package://rmcs_description/meshes/rmcs/collision/base_link.stl" /> -->
+          <!-- <mesh filename="package://rmcs_description/meshes/rmcs/collision/base_link.stl" /> -->
         </geometry>
       </collision>
     </link>
-    <!-- All-zero tool frame. This frame should correspond to the TOOL frame of the robot's controller.) -->
+    <!-- All-zero tool frame correspond to the TOOL frame of the robot's controller -->
     <link name="${prefix}tool0" />
     <!-- tool link -->
