Commit message: Add runtime display

File: rmcs_ws/src/rmcs_description/urdf/medium_feed_omni_wheel.xacro (robot description, xacro)
@@ -55,3 +55,21 @@
     <origin xyz="0 0 0" />
   </joint>
+  <link name="imu_link" />
+  <joint name="imu" type="fixed">
+    <parent link="pitch_link" />
+    <child link="imu_link" />
+    <origin rpy = "0 0 ${pi/2}" xyz="0 0 0" />
+  </joint>
+  <link name="muzzle_link" />
+  <joint name="muzzle" type="fixed">
+    <parent link="pitch_link" />
+    <child link="muzzle_link" />
+    <origin xyz="0.059 0 0" />
+  </joint>
+  <link name="camera_link" />
+  <joint name="camera" type="fixed">
+    <parent link="pitch_link" />
+    <child link="camera_link" />
+    <origin xyz="0.06603 0 0.082" />
+  </joint>
 </robot>

Commit message: Mamba out

File: rmcs_ws/src/rmcs_description/urdf/medium_feed_omni_wheel.xacro (robot description, xacro)
@@ -73,3 +73,27 @@
     <origin xyz="0.06603 0 0.082" />
   </joint>
+  <link name="omni_link_left_front" />
+  <joint name="omni" type="fixed">
+    <parent link="yaw_link" />
+    <child link="omni_link_left_front" />
+    <origin xyz="" />
+  </joint>
+  <link name="omni_link_right_front" />
+  <joint name="omni" type="fixed">
+    <parent link="yaw_link" />
+    <child link="omni_link_right_front" />
+    <origin xyz="" />
+  </joint>
+  <link name="omni_link_left" />
+  <joint name="omni" type="fixed">
+    <parent link="yaw_link" />
+    <child link="omni_link_left" />
+    <origin xyz="" />
+  </joint>
+  <link name="omni_link_right" />
+  <joint name="omni" type="fixed">
+    <parent link="yaw_link" />
+    <child link="omni_link_right" />
+    <origin xyz="" />
+  </joint>
 </robot>
