Commit message: Change default mode

File: rmcs_ws/src/rmcs_description/urdf/rmcs/rmcs_macro.xacro (robot description, xacro)
@@ -24,7 +24,4 @@
       </collision>
     </link>
-    <!-- All-zero tool frame correspond to the TOOL frame of the robot's controller -->
-    <link name="${prefix}tool0" />
-    <!-- tool link -->
     <!-- END LINKS -->
     <!-- JOINTS -->
